File: 4_Touch_Sensor_Board/4_Touch_Sensor_Board.kicad_sch (KiCad schematic)
At the start: 19 parts, among them J1 Conn_02x05, U1 TTP224B

Commit message: changes to upload
Parts:
- U1: footprint Package_SO:SSOP-16_3.9x4.9mm_P0.635mm -> (none)
Changed lines of the file:
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@@
     (pin "2")
   )
-  (symbol (lib_id "Touch_Sensor_CH:TTP224B") (at 146.685 85.725 0) (unit 1)
+  (symbol (lib_name "TTP224B_1") (lib_id "Touch_Sensor_CH:TTP224B") (at 146.685 85.725 0) (unit 1)
     (in_bom yes) (on_board yes)
-    (property "Reference" "U1" (id 0) (at 136.525 69.215 0)
-      (effects (font (size 1.27 1.27)) (justify left))
-    )
-    (property "Value" "TTP224B" (id 1) (at 136.525 71.755 0)
-      (effects (font (size 1.27 1.27)) (justify left))
-    )
-    (property "Footprint" "Package_SO:SSOP-16_3.9x4.9mm_P0.635mm" (id 2) (at 146.685 85.725 0)
+    (property "Reference" "U1" (id 0) (at 137.16 69.215 0)
+      (effects (font (size 1.27 1.27)) (justify left))
+    )
+    (property "Value" "TTP224B" (id 1) (at 137.16 71.755 0)
+      (effects (font (size 1.27 1.27)) (justify left))
+    )
+    (property "Footprint" "" (id 2) (at 146.685 85.725 0)
       (effects (font (size 0 0)) hide)
     )
@@
       (reference "R1") (unit 1) (value "330") (footprint "Resistor_SMD:R_0402_1005Metric")
     )
-    (path "/4e0182ac-968a-47f8-96a3-99709f8d98d6"
-      (reference "U1") (unit 1) (value "TTP224B") (footprint "Package_SO:SSOP-16_3.9x4.9mm_P0.635mm")
-    )
-  )
+    (path "/4bf82d12-eba8-4a68-9167-e5dca218a89b"
+      (reference "U1") (unit 1) (value "TTP224B") (footprint "")
+    )
+  )
